File: stm_audio_board_V3/Input_stage.kicad_sch (KiCad schematic)
At the start: 19 parts, among them U4 OP275

Commit message: Input and output stages are made and assembly started on pcb view
Parts:
- added C17 (x3), C18 (x3): 10p, Capacitor_SMD:C_0603_1608Metric, symbol Device:C_Small
- added C18 (x9): 100n, Capacitor_SMD:C_0603_1608Metric, symbol Device:C_Small
- added C19 (x3): 120p, Capacitor_SMD:C_0603_1608Metric, symbol Device:C_Small
- added C21 (x3), C23 (x3): 1nF, Capacitor_SMD:C_0603_1608Metric, symbol Device:C_Small
- added C24 (x3): 100pF, Capacitor_SMD:C_0603_1608Metric, symbol Device:C_Small
- added R4 (x9): 100R, Resistor_SMD:R_0603_1608Metric, symbol Device:R
- added R4 (x3), R5 (x3): 1M, Resistor_SMD:R_0603_1608Metric, symbol Device:R
- added R6 (x3), R7 (x3): 5.76k, Resistor_SMD:R_0603_1608Metric, symbol Device:R
- added R8 (x3), R9 (x3): 240R, Resistor_SMD:R_0603_1608Metric, symbol Device:R
- added U4 (x3): OP275, Package_SO:SSOP-8_3.9x5.05mm_P1.27mm, symbol Amplifier_Operational:OP275
- C17, C18, C19, C21, C23, C24: footprint Capacitor_SMD:C_0603_1608Metric_Pad1.08x0.95mm_HandSolder -> Capacitor_SMD:C_0603_1608Metric
- C18: value 68n -> 100n; footprint Capacitor_SMD:C_0603_1608Metric_Pad1.08x0.95mm_HandSolder -> Capacitor_SMD:C_0603_1608Metric
- R4, R5, R6, R7, R8, R9: footprint Resistor_SMD:R_0805_2012Metric_Pad1.20x1.40mm_HandSolder -> Resistor_SMD:R_0603_1608Metric
- R4: value 500k -> 1M; footprint Resistor_SMD:R_0805_2012Metric_Pad1.20x1.40mm_HandSolder -> Resistor_SMD:R_0603_1608Metric
- R4: value 100 -> 100R; footprint Resistor_SMD:R_0805_2012Metric_Pad1.20x1.40mm_HandSolder -> Resistor_SMD:R_0603_1608Metric
Connections:
- net ADC1N: now also C21.2, C21.2, C21.2, C24.2, C24.2, C24.2, R8.1, R8.1, R8.1
- net ADC1P: now also C23.1, C23.1, C23.1, C24.1, C24.1, C24.1, R9.1, R9.1, R9.1
- net GND: now also C18.1, C18.1, C18.1, C18.2, C18.2, C18.2, C18.2, C18.2, C18.2, C21.1, C21.1, C21.1, C23.2, C23.2, C23.2
- net VBIAS: now also R4.2, R4.2, R4.2, R4.2, R4.2, R4.2
- net GUITAR_IN renamed Audio_Main_Input
- new net: C18.1, R4.1, U4.3 (+) (x3)
- new net: C19.1, R6.1, R7.2, U4.6 (-) (x3)
- new net: C17.2, R5.1, R6.2, R8.2, U4.1 (x3)
- new net: C19.2, R7.1, R9.2, U4.7 (x3)
- new net: C17.1, R4.1, R5.2, U4.2 (-) (x3)
- new net: C18.1, R4.2 (x3)
- new net: C18.2, C18.2, R4.2 (x3)
- new net: C18.1, R4.1, U4.5 (+) (x3)
- new net Audio_Loop1_Return: R4.1
- new net Audio_Loop2_Return: R4.1
- new net Audio_Loop3_Return: R4.1
