File: stm_audio_board_V3/Input_stage.kicad_sch (KiCad schematic)
At the start: 92 parts, among them U4 OP275

Commit message: minor changes to components
Parts:
- C18: value 100n -> 100nF; JLCPCB (none) -> C14663; LCSC Part (none) -> C14663
- C18: value 10p -> 100pF; JLCPCB (none) -> C14858; LCSC Part (none) -> C14858
- C19: value 120p -> 100pF; JLCPCB (none) -> C14858; LCSC Part (none) -> C14858
- C21, C23: JLCPCB (none) -> C1588; LCSC Part (none) -> C1588
- C24: JLCPCB (none) -> C14858; LCSC Part (none) -> C14858
- D1, D12, D13, D14, D15, D16, D17, D18, D19, D20, D4, D5, D6, D7, D8, D9: JLCPCB (none) -> C191023; LCSC Part (none) -> C191023
- R4: JLCPCB (none) -> C22775; LCSC Part (none) -> C22775
- R4: JLCPCB (none) -> C22935; LCSC Part (none) -> C22935
- R5: value 1M -> 510k; JLCPCB (none) -> C23192; LCSC Part (none) -> C23192
- R6, R7: value 5.76k -> 4k7; JLCPCB (none) -> C23162; LCSC Part (none) -> C23162
- R8, R9: value 220R -> 100R; JLCPCB (none) -> C22775; LCSC Part (none) -> C22775
- U4: LCSC Part (none) -> C161797
