File: stm_audio_board_V3/stm_audio_board_V3.kicad_pcb (KiCad board)
At the start: 4 copper layers, 201 x 117 mm, 237 parts, among them J1 Power conn, J10 USB_A, J11 AudioJack_Loop1_Return, J12 AudioJack_Loop1_Send, J13 AudioJack_INPUT_Main, J14 AudioJack_OUTPUT_Main, J15 AudioJack_Loop2_Send, J2 STlink, J3 Audio_sig, J4 Conn_01x01_taptempo, J5 Barrel_Jack_MountingPin, J6 Conn_01x03_pot_ext, J7 AudioJack_Loop3_Return, J8 AudioJack_Loop3_Send, J9 AudioJack_Loop2_Return, SW1 SW_SPST, U1 IS42S16100H-7TL, U10 OP275, U12 OP275, U14 OP275, U2 OP275, U3 MP-K7805-500R3, U4 OP275, U5 MIC2920A-3.3WS-TR, U6 L7809, U7 STM32H723ZGTx, U8 OP275, U9 MIC2920A-3.3WS-TR, Y2 X1E0000210132

Commit message: Input output connected to codec
Parts:
- removed D4, D6, D8, D9: BAT42W-V, Diode_SMD:D_SOD-123
- removed H1, H2, H3, H4: MountingHole_Pad, MountingHole:MountingHole_3.2mm_M3_DIN965_Pad
- removed R18, R24, R66, R74: 10k, Resistor_SMD:R_0603_1608Metric
- added C120: 100n, Capacitor_SMD:C_0603_1608Metric, F.Cu at (113.2, 68.3)
- added C121: 100n, Capacitor_SMD:C_0603_1608Metric, F.Cu at (204.8, 70.8)
- added C122: 100n, Capacitor_SMD:C_0603_1608Metric, F.Cu at (225.2, 86.7)
- added RV1: R_Potentiometer, Potentiometer_THT:Potentiometer_Alps_RK09L_Single_Vertical, F.Cu at (150.5, 114.3)
- added RV2: R_Potentiometer, Potentiometer_THT:Potentiometer_Alps_RK09L_Single_Vertical, F.Cu at (169.1, 114.6)
- added RV3: R_Potentiometer, Potentiometer_THT:Potentiometer_Alps_RK09L_Single_Vertical, F.Cu at (187.6, 114.6)
- added RV4: R_Potentiometer, Potentiometer_THT:Potentiometer_Alps_RK09L_Single_Vertical, F.Cu at (150.5, 136.8)
- added RV5: R_Potentiometer, Potentiometer_THT:Potentiometer_Alps_RK09L_Single_Vertical, F.Cu at (169.1, 136.8)
- added RV6: R_Potentiometer, Potentiometer_THT:Potentiometer_Alps_RK09L_Single_Vertical, F.Cu at (187.6, 137.0)
- C113, C119, C43, C47: value 2.2nF -> 100n
- C20, C65, C87, C98: value 10p -> 1p
- R39, R40, R48, R49, R57, R58, R8, R9: value 240R -> 220R
- moved C119 141.1 mm to (257.9, 70.5), turned to -90 degrees
- moved C8 139.7 mm to (237.3, 106.4)
- moved C9 139.7 mm to (237.3, 108.9)
- moved C5 129.7 mm to (227.4, 100.6)
- moved C32 129.6 mm to (229.3, 93.2), turned to -90 degrees
- moved C25 128.5 mm to (231.1, 82.9), turned to 180 degrees
- moved C79 128.3 mm to (231.9, 93.9), turned to 180 degrees
- moved C80 127.7 mm to (234.3, 91.0)
- moved C26 124.1 mm to (231.4, 86.3)
- moved C6 118.0 mm to (215.1, 100.5), turned to 180 degrees
- moved C7 116.6 mm to (212.6, 97.7), turned to 180 degrees
- moved C34 113.7 mm to (211.7, 92.0), turned to 180 degrees
- moved C68 113.5 mm to (215.9, 86.1), turned to 90 degrees
- moved R10 106.5 mm to (213.5, 87.7)
- moved C67 106.0 mm to (213.2, 85.6)
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Connections:
- C101 pad 2: ADC1N -> ADC4N
- C106 pad 1: ADC1P -> ADC4P
- C107 pad 1: ADC1P -> ADC4P
- C107 pad 2: ADC1N -> ADC4N
- C112 pad 2: Audio_Loop2_Send -> Audio_Loop3_Send
- C113 pad 1: GND -> +9V
- C113 pad 2: Audio_Loop2_Send -> GND
- C118 pad 2: Audio_Loop3_Send -> Audio_Main_Output
- C119 pad 1: GND -> +9V
- C119 pad 2: Audio_Loop3_Send -> GND
- C42 pad 2: Audio_Main_Output -> Audio_Loop2_Send
- C43 pad 1: GND -> +9V
- C43 pad 2: Audio_Main_Output -> GND
- C47 pad 1: GND -> +9V
- C47 pad 2: Audio_Loop1_Send -> GND
- C74 pad 2: ADC1N -> ADC2N
- C82 pad 1: ADC1P -> ADC2P
- C83 pad 1: ADC1P -> ADC2P
- C83 pad 2: ADC1N -> ADC2N
- C92 pad 2: ADC1N -> ADC3N
- C93 pad 1: ADC1P -> ADC3P
- C94 pad 1: ADC1P -> ADC3P
- C94 pad 2: ADC1N -> ADC3N
- R15 pad 1: DAC1P -> DAC1N
- R16 pad 1: DAC1N -> DAC1P
- R27 pad 1: DAC1N -> DAC2P
- R30 pad 1: DAC1P -> DAC2N
- R39 pad 1: ADC1N -> ADC2N
- R40 pad 1: ADC1P -> ADC2P
- R48 pad 1: ADC1N -> ADC3N
- R49 pad 1: ADC1P -> ADC3P
- R57 pad 1: ADC1N -> ADC4N
- R58 pad 1: ADC1P -> ADC4P
- R59 pad 1: DAC1P -> DAC4P
- R60 pad 1: DAC1N -> DAC4N
- R67 pad 1: DAC1P -> DAC3N
- R68 pad 1: DAC1N -> DAC3P
- U11 pad 10: unconnected-(U11A-OL4P-Pad10) -> DAC4P
- U11 pad 11: unconnected-(U11A-OL4N-Pad11) -> DAC4N
- U11 pad 12: unconnected-(U11A-OR4P-Pad12) -> DAC3P
- U11 pad 13: unconnected-(U11A-OR4N-Pad13) -> DAC3N
- U11 pad 40: DAC1P -> unconnected-(U11A-OL2P-Pad40)
- U11 pad 41: DAC1N -> unconnected-(U11A-OL2N-Pad41)
- U11 pad 42: DAC2P -> unconnected-(U11A-OR2P-Pad42)
- U11 pad 43: DAC2N -> unconnected-(U11A-OR2N-Pad43)
- U11 pad 55: unconnected-(U11A-ADC1RP-Pad55) -> ADC2P
- U11 pad 56: unconnected-(U11A-ADC1RN-Pad56) -> ADC2N
- U11 pad 57: unconnected-(U11A-ADC2LP-Pad57) -> ADC3P
- U11 pad 58: unconnected-(U11A-ADC2LN-Pad58) -> ADC3N
- U11 pad 59: unconnected-(U11A-ADC2RP-Pad59) -> ADC4P
- U11 pad 6: unconnected-(U11A-OL3P-Pad6) -> DAC2P
- U11 pad 60: unconnected-(U11A-ADC2RN-Pad60) -> ADC4N
- U11 pad 7: unconnected-(U11A-OL3N-Pad7) -> DAC2N
- U11 pad 8: unconnected-(U11A-OR3P-Pad8) -> DAC1P
- U11 pad 9: unconnected-(U11A-OR3N-Pad9) -> DAC1N
- U14 pad 4: (no net) -> -9V
- U14 pad 8: (no net) -> +9V
Routing:
- net +9V: track 0.00 -> 245.3 mm, vias 0 -> 6
- net -9V: track 0.00 -> 231.9 mm, vias 0 -> 6
- net AD1939_CM: track 1.38 -> 216.2 mm, vias 1 -> 12
- net DAC3N: track 0.00 -> 121.6 mm, vias 0 -> 2
- net DAC3P: track 0.00 -> 118.9 mm, vias 0 -> 2
- net ADC4P: track 0.00 -> 106.5 mm
- net ADC4N: track 0.00 -> 106.5 mm
- net GND: track 1.61 -> 88.0 mm, vias 1 -> 58
- net DAC4P: track 0.00 -> 83.8 mm, vias 0 -> 2
- net DAC4N: track 0.00 -> 83.1 mm, vias 0 -> 2
- net ADC3N: track 0.00 -> 56.1 mm
- net ADC3P: track 0.00 -> 56.1 mm
- net Audio_Main_Output: track 0.00 -> 33.1 mm
- net Audio_Loop2_Send: track 0.00 -> 31.8 mm
- net ADC2P: track 0.00 -> 28.9 mm
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- added copper zone on In1.Cu, net GND
- added copper zone on In2.Cu, net GND

Commit message: minor changes
Parts:
- added C123: 10p, Capacitor_SMD:C_0603_1608Metric, F.Cu at (142.5, 88.3)
- added C124: 100n, Capacitor_SMD:C_0603_1608Metric, F.Cu at (142.5, 90.8)
- added C125: 10p, Capacitor_SMD:C_0603_1608Metric, F.Cu at (142.5, 93.3)
- added C126: 100n, Capacitor_SMD:C_0603_1608Metric, F.Cu at (155.7, 142.2)
- added C127: 100n, Capacitor_SMD:C_0603_1608Metric, F.Cu at (158.2, 142.2)
- added C128: 100n, Capacitor_SMD:C_0603_1608Metric, F.Cu at (160.7, 142.2)
- added C129: 100n, Capacitor_SMD:C_0603_1608Metric, F.Cu at (163.2, 142.2)
- added C130: 100n, Capacitor_SMD:C_0603_1608Metric, F.Cu at (165.7, 142.2)
- added C131: 100n, Capacitor_SMD:C_0603_1608Metric, F.Cu at (168.2, 142.2)
- added D2: LED, LED_SMD:LED_0603_1608Metric_Pad1.05x0.95mm_HandSolder, F.Cu at (142.7, 106.9)
- added D3: LED, LED_SMD:LED_0603_1608Metric_Pad1.05x0.95mm_HandSolder, F.Cu at (142.7, 109.5)
- added H1: MountingHole_Pad, MountingHole:MountingHole_3.2mm_M3_DIN965_Pad, F.Cu at (84.1, 78.8)
- added H2: MountingHole_Pad, MountingHole:MountingHole_3.2mm_M3_DIN965_Pad, F.Cu at (74.9, 142.9)
- added H3: MountingHole_Pad, MountingHole:MountingHole_3.2mm_M3_DIN965_Pad, F.Cu at (180.2, 143.6)
- added H4: MountingHole_Pad, MountingHole:MountingHole_3.2mm_M3_DIN965_Pad, F.Cu at (236.9, 73.2)
- added J16: STlink_DISP_MCU, Connector_PinHeader_2.54mm:PinHeader_1x04_P2.54mm_Vertical, F.Cu at (147.3, 85.0)
- added R18: 10k, Resistor_SMD:R_0603_1608Metric, F.Cu at (142.5, 95.8)
- added R24: 1k, Resistor_SMD:R_0603_1608Metric_Pad0.98x0.95mm_HandSolder, F.Cu at (137.0, 124.1)
- added R66: 1k, Resistor_SMD:R_0603_1608Metric_Pad0.98x0.95mm_HandSolder, F.Cu at (137.0, 126.6)
- added R74: 100R, Resistor_SMD:R_0603_1608Metric, F.Cu at (142.5, 98.3)
- added SW2: SW_SPST, Button_Switch_SMD:SW_SPST_TL3305A, F.Cu at (140.0, 114.4)
- added U15: STM32H723ZGTx, Package_QFP:LQFP-144_20x20mm_P0.5mm, F.Cu at (128.3, 99.2)
- added Y1: X1E0000210132, Crystal:Crystal_SMD_SeikoEpson_TSX3225-4Pin_3.2x2.5mm_HandSoldering, F.Cu at (138.1, 120.1)
- C121, C122: value 100n -> 2.2uF; footprint Capacitor_SMD:C_0603_1608Metric -> Capacitor_SMD:C_0805_2012Metric_Pad1.18x1.45mm_HandSolder
- J2: value STlink -> STlink_DSP
- moved J2 150.7 mm to (238.1, 111.0), turned to 180 degrees
- moved C122 84.2 mm to (142.9, 104.1)
- moved C121 69.0 mm to (142.9, 101.1)
- moved C28 22.0 mm to (241.6, 118.7)
- moved C9 10.5 mm to (247.8, 108.5)
- moved C29 10.5 mm to (248.9, 106.5)
- moved C8 10.5 mm to (247.8, 106.0)
- moved RV6 5.70 mm to (182.8, 134.0)
- moved C105 5.44 mm to (246.9, 88.0)
- moved C30 5.44 mm to (247.5, 100.5)
- moved C104 5.44 mm to (253.1, 88.0)
- moved C27 5.44 mm to (244.0, 88.0)
- moved FB4 5.44 mm to (249.9, 89.0)
- moved U5 5.44 mm to (248.5, 95.8)
- moved RV3 5.34 mm to (182.5, 116.0)
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Connections:
- C121 pad 1: +9V -> Net-(C121-Pad1)
- C122 pad 1: +3.3VA -> Net-(C122-Pad1)
- J2 pad 2: SWDIO -> SWDIO_DSP
- J2 pad 3: SWCLK -> SWCLK_DSP
- RV1 pad 1: unconnected-(RV1-Pad1) -> +3.3V
- RV1 pad 2: unconnected-(RV1-Pad2) -> POT1
- RV1 pad 3: unconnected-(RV1-Pad3) -> GND
- RV2 pad 1: unconnected-(RV2-Pad1) -> +3.3V
- RV2 pad 2: unconnected-(RV2-Pad2) -> POT2
- RV2 pad 3: unconnected-(RV2-Pad3) -> GND
- RV3 pad 1: unconnected-(RV3-Pad1) -> +3.3V
- RV3 pad 2: unconnected-(RV3-Pad2) -> POT3
- RV3 pad 3: unconnected-(RV3-Pad3) -> GND
- RV4 pad 1: unconnected-(RV4-Pad1) -> +3.3V
- RV4 pad 2: unconnected-(RV4-Pad2) -> POT4
- RV4 pad 3: unconnected-(RV4-Pad3) -> GND
- RV5 pad 1: unconnected-(RV5-Pad1) -> +3.3V
- RV5 pad 2: unconnected-(RV5-Pad2) -> POT5
- RV5 pad 3: unconnected-(RV5-Pad3) -> GND
- RV6 pad 1: unconnected-(RV6-Pad1) -> +3.3V
- RV6 pad 2: unconnected-(RV6-Pad2) -> POT6
- RV6 pad 3: unconnected-(RV6-Pad3) -> GND
- U11 pad 19: AD1939_I2S2_SDO -> unconnected-(U11A-DSDATA2-Pad19)
- U11 pad 20: unconnected-(U11A-DSDATA1-Pad20) -> AD1939_SAI1A_SDO
- U11 pad 21: AD1939_I2S2_CK -> AD1939_SAI1A_CK
- U11 pad 22: AD1939_I2S2_WS -> AD1939_SAI1A_WS
- U11 pad 27: AD1939_I2S1_SDI -> AD1939_SAI1B_SDI
- U11 pad 28: AD1939_I2S1_CK -> AD1939_SAI1A_CK
- U11 pad 29: AD1939_I2S1_WS -> AD1939_SAI1A_WS
- U14 pad 4: -9V -> (no net)
- U14 pad 8: +9V -> (no net)
- U7 pad 105: unconnected-(U7-PA13(JTMS-Pad105) -> SWDIO_DSP
- U7 pad 109: unconnected-(U7-PA14(JTCK-Pad109) -> SWCLK_DSP
- U7 pad 111: AD1939_I2S2_CK -> unconnected-(U7-PC10-Pad111)
- U7 pad 13: POT1 -> unconnected-(U7-PF3-Pad13)
- U7 pad 15: POT2 -> unconnected-(U7-PF5-Pad15)
- U7 pad 19: POT3 -> unconnected-(U7-PF7-Pad19)
- U7 pad 2: unconnected-(U7-PE3-Pad2) -> AD1939_SAI1B_SDI
- U7 pad 20: POT4 -> unconnected-(U7-PF8-Pad20)
- U7 pad 21: POT5 -> unconnected-(U7-PF9-Pad21)
- U7 pad 22: POT6 -> unconnected-(U7-PF10-Pad22)
- U7 pad 28: AD1939_I2S1_SDI -> unconnected-(U7-PC2_C-Pad28)
- U7 pad 3: unconnected-(U7-PE4-Pad3) -> AD1939_SAI1A_WS
- U7 pad 4: unconnected-(U7-PE5-Pad4) -> AD1939_SAI1A_CK
- U7 pad 40: AD1939_I2S2_WS -> unconnected-(U7-PA4-Pad40)
- U7 pad 41: AD1939_SPI3_CLK -> unconnected-(U7-PA5-Pad41)
- U7 pad 42: AD1939_SPI3_MISO -> unconnected-(U7-PA6-Pad42)
- U7 pad 43: AD1939_SPI3_MOSI -> unconnected-(U7-PA7-Pad43)
- U7 pad 48: AD1939_I2S2_SDO -> unconnected-(U7-PB2-Pad48)
- U7 pad 5: unconnected-(U7-PE6-Pad5) -> AD1939_SAI1A_SDO
- U7 pad 69: AD1939_I2S1_CK -> unconnected-(U7-PB10-Pad69)
- U7 pad 73: AD1939_I2S1_WS -> unconnected-(U7-PB12-Pad73)
Routing:
- net SWCLK_DSP: track 0.00 -> 7.52 mm
- net SWDIO_DSP: track 0.00 -> 5.24 mm
