File: stm_audio_board_V3/stm_audio_board_V3.kicad_pcb (KiCad board)
At the start: 4 copper layers, 230.9 x 117 mm, 307 parts, among them J1 Power conn, J10 USB_A, J11 AudioJack_Loop1_Return, J12 AudioJack_Loop1_Send, J13 AudioJack_INPUT_Main, J14 AudioJack_OUTPUT_Main, J15 AudioJack_Loop2_Send, J16 STlink_DISP_MCU, J2 STlink_DSP, J3 Audio_sig, J4 Conn_01x01_taptempo, J5 Barrel_Jack_MountingPin, J6 Conn_01x03_pot_ext, J7 AudioJack_Loop3_Return, J8 AudioJack_Loop3_Send, J9 AudioJack_Loop2_Return, SW1 SW_SPST, SW2 SW_SPST, U1 IS42S16100H-7TL, U10 OP275, U12 OP275, U13 LM7809_TO220, U14 OP275, U15 STM32H723ZGTx, U16 LM7909_TO220, U2 OP275, U3 7909, U4 OP275, U5 MIC2920A-3.3WS-TR, U6 7809, U7 STM32H723ZGTx, U8 OP275, U9 MIC2920A-3.3WS-TR, Y1 X1E0000210132, Y2 X1E0000210132

Commit message: Footswitch debounce added
Parts:
- removed C63: 100n, Capacitor_SMD:C_0603_1608Metric
- removed U16: LM7909_TO220, Package_TO_SOT_THT:TO-220-3_Vertical
- added C174: 100n, Capacitor_SMD:C_0603_1608Metric, F.Cu at (204.8, 78.3)
- added C175: 100n, Capacitor_SMD:C_0603_1608Metric, F.Cu at (251.9, 63.5)
- added C176: 100n, Capacitor_SMD:C_0603_1608Metric, F.Cu at (102.9, 63.9)
- added C177: 100n, Capacitor_SMD:C_0603_1608Metric, F.Cu at (152.9, 63.3)
- added C178: 100n, Capacitor_SMD:C_0603_1608Metric, F.Cu at (203.6, 64.4)
- added C179: 100n, Capacitor_SMD:C_0603_1608Metric, F.Cu at (111.1, 69.0)
- added C180: 100n, Capacitor_SMD:C_0603_1608Metric, F.Cu at (103.6, 76.9)
- added C181: 100n, Capacitor_SMD:C_0603_1608Metric, F.Cu at (202.2, 110.8)
- added C182: 100n, Capacitor_SMD:C_0603_1608Metric, F.Cu at (220.7, 130.4)
- added C183: 100n, Capacitor_SMD:C_0603_1608Metric, F.Cu at (206.2, 129.7)
- added C184: 100n, Capacitor_SMD:C_0603_1608Metric, F.Cu at (152.5, 116.4)
- added C185: 100n, Capacitor_SMD:C_0603_1608Metric, F.Cu at (184.5, 123.8)
- added C186: 100n, Capacitor_SMD:C_0603_1608Metric, F.Cu at (184.6, 126.9)
- added C187: 100n, Capacitor_SMD:C_0603_1608Metric, F.Cu at (184.6, 130.5)
- added C188: 100n, Capacitor_SMD:C_0603_1608Metric, F.Cu at (193.7, 130.3)
- added C189: 100n, Capacitor_SMD:C_0603_1608Metric, F.Cu at (191.4, 123.0)
- added J17: Conn_01x10_Footswitch, Connector_IDC:IDC-Header_2x05_P2.54mm_Vertical, F.Cu at (181.1, 143.7)
- added R75: 10k, Resistor_SMD:R_0603_1608Metric_Pad0.98x0.95mm_HandSolder, F.Cu at (182.0, 124.5)
- added R76: 1k, Resistor_SMD:R_0603_1608Metric_Pad0.98x0.95mm_HandSolder, F.Cu at (182.1, 122.8)
- added R77: 1k, Resistor_SMD:R_0603_1608Metric_Pad0.98x0.95mm_HandSolder, F.Cu at (182.0, 127.7)
- added R78: 10k, Resistor_SMD:R_0603_1608Metric_Pad0.98x0.95mm_HandSolder, F.Cu at (182.0, 126.1)
- added R79: 1k, Resistor_SMD:R_0603_1608Metric_Pad0.98x0.95mm_HandSolder, F.Cu at (182.1, 131.3)
- added R80: 10k, Resistor_SMD:R_0603_1608Metric_Pad0.98x0.95mm_HandSolder, F.Cu at (182.1, 129.7)
- added R81: 1k, Resistor_SMD:R_0603_1608Metric_Pad0.98x0.95mm_HandSolder, F.Cu at (194.7, 132.6)
- added R82: 10k, Resistor_SMD:R_0603_1608Metric_Pad0.98x0.95mm_HandSolder, F.Cu at (196.2, 131.1)
- added R83: 1k, Resistor_SMD:R_0603_1608Metric_Pad0.98x0.95mm_HandSolder, F.Cu at (191.5, 135.6)
- added R84: 1k, Resistor_SMD:R_0603_1608Metric_Pad0.98x0.95mm_HandSolder, F.Cu at (187.8, 135.6)
- added R85: 1k, Resistor_SMD:R_0603_1608Metric_Pad0.98x0.95mm_HandSolder, F.Cu at (189.6, 135.6)
- L1, L2, L3, L4, L5, L6, L7, L8: footprint Inductor_SMD:L_6.3x6.3_H3 -> Inductor_SMD:L_Sunlord_SWPA6020S
- R33: value 500k -> 1k; footprint Resistor_SMD:R_0805_2012Metric_Pad1.20x1.40mm_HandSolder -> Resistor_SMD:R_0603_1608Metric_Pad0.98x0.95mm_HandSolder
- U13: value LM7809_TO220 -> 74HC14; footprint Package_TO_SOT_THT:TO-220-3_Vertical -> Package_SO:SOIC-14_3.9x8.7mm_P1.27mm
- U9: footprint Package_TO_SOT_SMD:SOT-223-3_TabPin2 -> Package_TO_SOT_SMD:SOT-89-3
- moved U13 113.5 mm to (189.1, 128.5), turned to 0 degrees
- moved C14 113.4 mm to (229.0, 109.3), turned to -90 degrees
- moved C3 110.7 mm to (229.0, 120.6), turned to -90 degrees
- moved C10 108.5 mm to (208.6, 104.5)
- moved C12 106.3 mm to (219.5, 104.6)
- moved C36 105.7 mm to (227.2, 133.3), turned to -90 degrees
- moved C58 102.7 mm to (228.3, 128.3), turned to 90 degrees
- moved C11 101.2 mm to (214.9, 104.5)
- moved C43 99.9 mm to (211.4, 70.5), turned to 180 degrees
- moved C113 99.8 mm to (111.7, 56.2), turned to 90 degrees
- moved C119 99.8 mm to (161.0, 55.9), turned to 90 degrees
- moved C120 99.1 mm to (211.5, 56.1), turned to 90 degrees
- moved C47 98.1 mm to (260.1, 56.2), turned to 90 degrees
- moved C35 96.0 mm to (215.9, 129.6), turned to 180 degrees
- moved C60 87.2 mm to (203.6, 121.5), turned to -90 degrees
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Connections:
- R33 pad 1: EXT_INT_BUTTON -> LED1_PIN
- R33 pad 2: TAP_TEMPO_INPUT -> LED1
- U13 pad 1: unconnected-(U13-VI-Pad1) -> Net-(C185-Pad1)
- U13 pad 2: GND -> Footswitch_1_INTERRUPT_PIN
- U13 pad 3: unconnected-(U13-VO-Pad3) -> Net-(C186-Pad1)
- U14 pad 4: (no net) -> -9V
- U14 pad 8: (no net) -> +9V
Routing:
- net +3.3V: track 10.6 -> 90.6 mm, vias 0 -> 3
- net +9V: track 205.6 -> 264.7 mm
- net ADC1P: track 6.15 -> 63.5 mm
- net ADC1N: track 6.32 -> 62.5 mm
- net GND: track 108.7 -> 154.9 mm, vias 234 -> 274
- net Footswitch_2: track 0.00 -> 24.1 mm, vias 0 -> 1
- net PWR_INPUT_12V-18V: track 23.3 -> 0.00 mm
- net Footswitch_4: track 0.00 -> 23.2 mm
- net /Power/+12V: track 20.6 -> 0.02 mm
- net Footswitch_1: track 0.00 -> 20.1 mm
- net AD1939_CM: track 197.1 -> 217.0 mm, vias 10 -> 9
- net /Power/-12V: track 18.8 -> 0.00 mm
- net AD1939_SAI1A_CK: track 0.00 -> 15.8 mm
- net AD1939_SAI1A_WS: track 0.00 -> 15.7 mm, vias 0 -> 2
- net LED2: track 0.00 -> 15.5 mm
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- added copper zone on F.Cu, net /Power/+12V
- added copper zone on F.Cu, net /Power/-12V
- added copper zone on F.Cu, net Net-(PS2-+Vin)
- added copper zone on F.Cu, net Net-(U6-IN)
- removed copper zone on F.Cu, net unconnected-(U13-VI-Pad1)

Commit message: USB added
Parts:
- added J18: USB3_A, Connector_USB:USB3_A_Receptacle_Wuerth_692122030100, F.Cu at (242.8, 148.9)
- moved H4 244.2 mm to (73.6, 143.6)
- moved D11 94.5 mm to (168.9, 170.2)
- moved C59 75.9 mm to (87.0, 111.6), turned to 180 degrees
- moved C151 69.3 mm to (248.5, 105.6), turned to -90 degrees
- moved C160 68.9 mm to (265.1, 107.4), turned to -90 degrees
- moved L6 67.4 mm to (260.5, 100.5)
- moved C148 67.4 mm to (256.9, 106.6)
- moved C149 67.4 mm to (260.6, 106.6)
- moved C157 67.4 mm to (254.1, 106.6)
- moved C158 67.4 mm to (263.0, 106.6)
- moved D10 66.7 mm to (182.2, 168.3)
- moved R12 66.7 mm to (173.0, 166.8)
- moved R25 66.7 mm to (173.0, 169.3)
- moved C140 66.2 mm to (245.8, 101.4), turned to 90 degrees
- moved H2 63.8 mm to (42.1, 88.2)
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Connections:
- U7 pad 102: unconnected-(U7-PA10-Pad102) -> DSP_USB_HS_ID
- U7 pad 103: unconnected-(U7-PA11-Pad103) -> DSP_USB_HS_DM
- U7 pad 104: unconnected-(U7-PA12-Pad104) -> DSP_USB_HS_DP
Routing:
- net DSP_USB_HS_DP: track 0.00 -> 38.5 mm
- net DSP_USB_HS_DM: track 0.00 -> 36.6 mm
- net /MCU/NRST: track 0.00 -> 33.3 mm
- net +3.3V: track 90.6 -> 114.6 mm
- net Net-(PS1-+Vout): track 14.5 -> 9.22 mm
- net 5V: track 8.19 -> 5.34 mm
- net GND: track 154.9 -> 153.7 mm, vias 274 -> 279
