File: stm_audio_board_V3/_autosave-stm_audio_board_V3.kicad_pcb (KiCad board)
At the start: 4 copper layers, 265 x 117 mm, 377 parts, among them J1 Power conn, J10 USB_A, J11 AudioJack_LOOP3_SEND, J12 AudioJack_LOOP3_RETURN, J13 AudioJack_OUTPUT, J14 AudioJack_INPUT, J15 AudioJack_LOOP2_RETURN, J16 STlink_DISP_MCU, J17 Conn_01x10_Footswitch, J18 Conn_01x16_ILI9341, J2 STlink_DSP, J3 Audio_sig, J4 Conn_01x01_taptempo, J5 Barrel_Jack_MountingPin, J6 Conn_01x03_pot_ext, J7 AudioJack_LOOP1_SEND, J8 AudioJack_LOOP1_RETURN, J9 AudioJack_LOOP2_SEND, SW1 SW_SPST, SW2 SW_SPST, U1 IS42S16100H-7TL, U10 OP275, U12 OP275, U13 74HC14, U14 OP275, U15 STM32H723ZGTx, U16 USBLC6-2P6, U17 W25Q128JVS, U18 W25Q128JVS, U19 FE1.1s, U2 OP275, U3 7909, U4 OP275, U5 MIC2920A-3.3WS-TR, U6 7809, U7 STM32H723ZGTx, U8 OP275, U9 MIC2920A-3.3WS-TR, Y1 X1E0000210132, Y2 X1E0000210132, Y3 Crystal_GND24

Commit message: 1117 regulator added
Parts:
- removed C89, C90: 100n, Capacitor_SMD:C_0603_1608Metric
- removed J1: Power conn, Connector_PinHeader_2.54mm:PinHeader_1x02_P2.54mm_Vertical
- removed J3: Audio_sig, Connector_PinHeader_2.54mm:PinHeader_1x03_P2.54mm_Vertical
- removed J4: Conn_01x01_taptempo, Connector_PinHeader_2.54mm:PinHeader_1x01_P2.54mm_Vertical
- removed J6: Conn_01x03_pot_ext, Connector_PinHeader_2.54mm:PinHeader_1x03_P2.54mm_Vertical
- removed U9: MIC2920A-3.3WS-TR, Package_TO_SOT_SMD:SOT-89-3
- added C205: 10uF, Capacitor_SMD:C_1206_3216Metric, F.Cu at (229.6, 99.2)
- added C206: 10uF, Capacitor_SMD:C_1206_3216Metric, F.Cu at (229.6, 101.8)
- added C207: 100n, Capacitor_SMD:C_0603_1608Metric, F.Cu at (223.5, 120.2)
- added C208: 100uf, Capacitor_THT:CP_Radial_D6.3mm_P2.50mm, F.Cu at (227.4, 123.0)
- added C209: 10uF, Capacitor_SMD:C_1206_3216Metric, F.Cu at (239.8, 102.5)
- added C210: 10uF, Capacitor_SMD:C_1206_3216Metric, F.Cu at (239.8, 99.9)
- added C211: 10uF, Capacitor_SMD:C_1206_3216Metric, F.Cu at (234.9, 97.3)
- added C212: 10uF, Capacitor_SMD:C_1206_3216Metric, F.Cu at (234.9, 99.9)
- added C213: 10uF, Capacitor_SMD:C_1206_3216Metric, F.Cu at (234.9, 102.5)
- added C214: 10uF, Capacitor_SMD:C_1206_3216Metric, F.Cu at (222.7, 124.7)
- added C215: 10uF, Capacitor_SMD:C_1206_3216Metric, F.Cu at (222.7, 122.2)
- added C216: 10uF, Capacitor_SMD:C_1206_3216Metric, F.Cu at (231.6, 116.6)
- added U20: AP1117-33, Package_TO_SOT_SMD:SOT-223-3_TabPin2, F.Cu at (224.3, 114.9)
- C29: value 47uF -> 100uf
- C4: value 100uF -> 10uF; footprint Capacitor_THT:CP_Radial_D6.3mm_P2.50mm -> Capacitor_SMD:C_1206_3216Metric
- C71: value 47uf -> 10uF; footprint Capacitor_THT:CP_Radial_D6.3mm_P2.50mm -> Capacitor_SMD:C_1206_3216Metric
- U5: value MIC2920A-3.3WS-TR -> AP1117-33
- moved C192 89.3 mm to (217.5, 125.9), turned to 180 degrees
- moved R1 79.2 mm to (211.8, 120.9), turned to -90 degrees
- moved C122 49.1 mm to (168.3, 96.7), turned to 90 degrees
- moved C71 45.9 mm to (234.1, 116.6), turned to 90 degrees
- moved TP6 25.3 mm to (251.1, 85.8)
- moved U5 24.1 mm to (231.0, 91.6), turned to 90 degrees
- moved C30 22.9 mm to (230.4, 97.0), turned to 180 degrees
- moved C4 19.4 mm to (239.8, 97.3), turned to 180 degrees
- moved C70 19.3 mm to (239.0, 118.1), turned to 90 degrees
- moved C102 16.2 mm to (229.6, 117.4), turned to 90 degrees
- moved C29 15.7 mm to (223.3, 101.1), turned to 90 degrees
- moved TP2 13.4 mm to (249.2, 96.0)
- moved C15 12.3 mm to (231.2, 107.1), turned to 180 degrees
- moved D11 9.65 mm to (162.8, 141.2)
- moved R12 9.46 mm to (166.2, 142.9)
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Connections:
- C71 pad 1: +3.3V -> 5V
- U5 pad 1: Net-(U5-VI) -> GND
- U5 pad 2: GND -> +3.3VA
- U5 pad 3: +3.3VA -> Net-(U5-VI)
Routing:
- net 5V: track 5.34 -> 46.3 mm
- net +3.3VA: track 70.4 -> 108.8 mm, vias 7 -> 8
- net +3.3V: track 422.2 -> 457.7 mm, vias 6 -> 7
- net GND: track 226.7 -> 243.7 mm, vias 377 -> 408
- net Net-(U5-VI): track 0.00 -> 16.2 mm
- net Net-(C122-Pad1): track 0.00 -> 4.72 mm
- net DISPLAY_USB_HS_D-: track 131.7 -> 134.4 mm
- net SWDIO_DISP: track 15.2 -> 17.8 mm
- net Net-(U7-BOOT0): track 0.00 -> 2.17 mm
- net DSP_USB_HS_D-: track 152.2 -> 154.0 mm
- added copper zone on F.Cu, net +3.3VA
