File: stm_audio_board_V3/_autosave-stm_audio_board_V3.kicad_pcb (KiCad board)
At the start: 4 copper layers, 265 x 117 mm, 398 parts, among them J10 USB_A, J11 AudioJack_LOOP3_SEND, J12 AudioJack_LOOP3_RETURN, J13 AudioJack_OUTPUT, J14 AudioJack_INPUT, J15 AudioJack_LOOP2_RETURN, J16 STlink_DISP_MCU, J17 Conn_01x10_Footswitch, J18 Conn_01x16_ILI9341, J2 STlink_DSP, J5 Barrel_Jack_MountingPin, J7 AudioJack_LOOP1_SEND, J8 AudioJack_LOOP1_RETURN, J9 AudioJack_LOOP2_SEND, SW1 SW_SPST, SW2 SW_SPST, U1 IS42S16100H-7TL, U10 OP275, U12 OP275, U13 74HC14, U14 OP275, U15 STM32H723ZGTx, U16 USBLC6-2P6, U17 W25Q128JVS, U18 W25Q128JVS, U19 FE1.1s, U2 OP275, U20 AP1117-33, U3 7909, U4 OP275, U5 AP1117-33, U6 7809, U7 STM32H723ZGTx, U8 OP275, U9 AP1117-33, Y1 X1E0000210132, Y2 X1E0000210132, Y3 Crystal_GND24

Commit message: added external pot, added feedback leds, added I2C between MCUs
Parts:
- removed D10, D11, D2, D3: LED, LED_SMD:LED_0603_1608Metric_Pad1.05x0.95mm_HandSolder
- removed the J14 at (56.6, 82.3)
- removed R66: 1k, Resistor_SMD:R_0603_1608Metric_Pad0.98x0.95mm_HandSolder
- added C227: 100n, Capacitor_SMD:C_0603_1608Metric, F.Cu at (186.8, 106.7)
- added DISPLAY_OK1: LED, LED_SMD:LED_0603_1608Metric_Pad1.05x0.95mm_HandSolder, F.Cu at (138.0, 98.3)
- added DSP_OK1: LED, LED_SMD:LED_0603_1608Metric_Pad1.05x0.95mm_HandSolder, F.Cu at (197.3, 143.9)
- added H5: MountingHole_Pad, MountingHole:MountingHole_3.2mm_M3_DIN965_Pad, F.Cu at (298.5, 104.8)
- added H6: MountingHole_Pad, MountingHole:MountingHole_3.2mm_M3_DIN965_Pad, F.Cu at (298.5, 54.5)
- added J1: External_POT, Connector_Audio:Jack_6.35mm_Neutrik_NMJ6HCD2_Horizontal, F.Cu at (60.3, 81.1)
- R24: value 1k -> 220R; footprint Resistor_SMD:R_0603_1608Metric_Pad0.98x0.95mm_HandSolder -> Resistor_SMD:R_0603_1608Metric
- moved R12 69.6 mm to (138.9, 100.9), turned to -90 degrees
- moved R24 66.7 mm to (184.4, 107.5), turned to 180 degrees
- moved TP7 48.8 mm to (235.8, 121.5)
- moved H1 47.2 mm to (171.8, 46.6)
- moved R25 37.9 mm to (196.3, 142.3)
- moved H2 22.1 mm to (48.5, 54.5)
- moved H4 15.6 mm to (48.5, 104.5)
- moved C100 6.16 mm to (81.2, 59.5)
- moved C95 6.16 mm to (68.1, 60.1)
- moved C96 6.16 mm to (68.1, 58.5)
- moved C98 6.16 mm to (72.0, 57.7)
- moved R50 6.16 mm to (68.1, 61.7)
- moved R52 6.16 mm to (71.1, 61.7)
- moved R53 6.16 mm to (70.4, 57.7)
- moved R55 6.16 mm to (81.1, 62.7)
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Connections:
- J12 pad TN: unconnected-(J12-PadTN) -> GND
- J14 pad TN: unconnected-(J14-PadTN) -> GND
- J15 pad TN: unconnected-(J15-PadTN) -> GND
- J8 pad TN: unconnected-(J8-PadTN) -> GND
- R12 pad 2: LED1 -> DISPLAY_OK_LED
- R24 pad 1: Net-(D3-A) -> EXT_POT_ADC
- R24 pad 2: LED1 -> Net-(J1-PadR)
- R25 pad 2: LED2 -> DSP_OK_LED
- U15 pad 100: unconnected-(U15-PA8-Pad100) -> I2C_SCL
- U15 pad 8: unconnected-(U15-PC14-Pad8) -> DISPLAY_OK_LED
- U15 pad 99: unconnected-(U15-PC9-Pad99) -> I2C_SDA
- U7 pad 36: unconnected-(U7-PA2-Pad36) -> EXT_POT_ADC
- U7 pad 81: unconnected-(U7-PD12-Pad81) -> I2C_SCL
- U7 pad 82: unconnected-(U7-PD13-Pad82) -> I2C_SDA
- U7 pad 90: unconnected-(U7-PG5-Pad90) -> DSP_OK_LED
Routing:
- net Net-(J1-PadR): track 0.00 -> 152.9 mm
- net I2C_SDA: track 0.00 -> 72.7 mm, vias 0 -> 2
- net I2C_SCL: track 0.00 -> 70.1 mm, vias 0 -> 2
- net +3.3V: track 869.3 -> 896.4 mm
- net EXT_POT_ADC: track 0.00 -> 11.5 mm
- net DSP_OK_LED: track 0.00 -> 7.10 mm
- net AD1939_CM: track 263.3 -> 257.3 mm
- net +9V: track 271.6 -> 265.6 mm
- net -9V: track 287.9 -> 282.1 mm
- net DISPLAY_OK_LED: track 0.00 -> 4.03 mm
- net POT6: track 123.2 -> 126.7 mm
- net ADC4N: track 153.4 -> 150.1 mm
- net ADC4P: track 153.5 -> 150.1 mm
- net POT3: track 135.6 -> 138.6 mm
- net POT4: track 49.6 -> 51.7 mm
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Other:
- board text added: "IN"
- board text added: "OUT"
