File: stm_audio_board_V3/Audio_Connectors.kicad_sch (KiCad schematic)
At the start: 8 parts, among them J12 AudioJack_LOOP2_RETURN, J13 AudioJack_LOOP3_RETURN, J14 AudioJack_INPUT, J15 AudioJack_LOOP1_SEND, J16 AudioJack_LOOP2_SEND, J7 AudioJack_LOOP1_RETURN, J8 AudioJack_LOOP3_SEND, J9 AudioJack_OUTPUT

Commit message: added silkscreen captions, capacitor between gnd and earth
Parts:
- J12, J13, J14, J15, J16, J7, J8, J9: footprint Connector_Audio:Jack_6.35mm_Neutrik_NMJ6HCD2_Horizontal -> stm_audio_board_footprints:6.3_jack_new_ref; LCSC Part C309275 -> C309277
Changed lines of the file:
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@@
       (effects (font (size 1.27 1.27)))
     )
-    (property "Footprint" "Connector_Audio:Jack_6.35mm_Neutrik_NMJ6HCD2_Horizontal" (at 92.71 147.32 0)
+    (property "Footprint" "stm_audio_board_footprints:6.3_jack_new_ref" (at 92.71 147.32 0)
       (effects (font (size 1.27 1.27)) hide)
     )
@@
       (effects (font (size 1.27 1.27)) hide)
     )
-    (property "LCSC Part" "C309275" (at 92.71 147.32 0)
+    (property "LCSC Part" "C309277" (at 92.71 147.32 0)
       (effects (font (size 1.27 1.27)) hide)
     )
@@
       (effects (font (size 1.27 1.27)))
     )
-    (property "Footprint" "Connector_Audio:Jack_6.35mm_Neutrik_NMJ6HCD2_Horizontal" (at 92.71 97.79 0)
+    (property "Footprint" "stm_audio_board_footprints:6.3_jack_new_ref" (at 92.71 97.79 0)
       (effects (font (size 1.27 1.27)) hide)
     )
@@
       (effects (font (size 1.27 1.27)) hide)
     )
-    (property "LCSC Part" "C309275" (at 92.71 97.79 0)
+    (property "LCSC Part" "C309277" (at 92.71 97.79 0)
       (effects (font (size 1.27 1.27)) hide)
     )
@@
       (effects (font (size 1.27 1.27)))
     )
-    (property "Footprint" "Connector_Audio:Jack_6.35mm_Neutrik_NMJ6HCD2_Horizontal" (at 40.64 38.1 0)
+    (property "Footprint" "stm_audio_board_footprints:6.3_jack_new_ref" (at 40.64 38.1 0)
       (effects (font (size 1.27 1.27)) hide)
     )
@@
       (effects (font (size 1.27 1.27)) hide)
     )
-    (property "LCSC Part" "C309275" (at 40.64 38.1 0)
+    (property "LCSC Part" "C309277" (at 40.64 38.1 0)
       (effects (font (size 1.27 1.27)) hide)
     )
@@
       (effects (font (size 1.27 1.27)))
     )
-    (property "Footprint" "Connector_Audio:Jack_6.35mm_Neutrik_NMJ6HCD2_Horizontal" (at 43.18 121.92 0)
+    (property "Footprint" "stm_audio_board_footprints:6.3_jack_new_ref" (at 43.18 121.92 0)
       (effects (font (size 1.27 1.27)) hide)
     )
@@
       (effects (font (size 1.27 1.27)) hide)
     )
-    (property "LCSC Part" "C309275" (at 43.18 121.92 0)
+    (property "LCSC Part" "C309277" (at 43.18 121.92 0)
       (effects (font (size 1.27 1.27)) hide)
     )
@@
       (effects (font (size 1.27 1.27)))
     )
-    (property "Footprint" "Connector_Audio:Jack_6.35mm_Neutrik_NMJ6HCD2_Horizontal" (at 90.17 38.1 0)
+    (property "Footprint" "stm_audio_board_footprints:6.3_jack_new_ref" (at 90.17 38.1 0)
       (effects (font (size 1.27 1.27)) hide)
     )
@@
       (effects (font (size 1.27 1.27)) hide)
     )
-    (property "LCSC Part" "C309275" (at 90.17 38.1 0)
+    (property "LCSC Part" "C309277" (at 90.17 38.1 0)
       (effects (font (size 1.27 1.27)) hide)
     )
@@
       (effects (font (size 1.27 1.27)))
     )
-    (property "Footprint" "Connector_Audio:Jack_6.35mm_Neutrik_NMJ6HCD2_Horizontal" (at 92.71 121.92 0)
+    (property "Footprint" "stm_audio_board_footprints:6.3_jack_new_ref" (at 92.71 121.92 0)
       (effects (font (size 1.27 1.27)) hide)
     )
@@
       (effects (font (size 1.27 1.27)) hide)
     )
-    (property "LCSC Part" "C309275" (at 92.71 121.92 0)
+    (property "LCSC Part" "C309277" (at 92.71 121.92 0)
       (effects (font (size 1.27 1.27)) hide)
     )
@@
       (effects (font (size 1.27 1.27)))
     )
-    (property "Footprint" "Connector_Audio:Jack_6.35mm_Neutrik_NMJ6HCD2_Horizontal" (at 43.18 97.79 0)
+    (property "Footprint" "stm_audio_board_footprints:6.3_jack_new_ref" (at 43.18 97.79 0)
       (effects (font (size 1.27 1.27)) hide)
     )
@@
       (effects (font (size 1.27 1.27)) hide)
     )
-    (property "LCSC Part" "C309275" (at 43.18 97.79 0)
+    (property "LCSC Part" "C309277" (at 43.18 97.79 0)
       (effects (font (size 1.27 1.27)) hide)
     )
@@
       (effects (font (size 1.27 1.27)))
     )
-    (property "Footprint" "Connector_Audio:Jack_6.35mm_Neutrik_NMJ6HCD2_Horizontal" (at 43.18 147.32 0)
+    (property "Footprint" "stm_audio_board_footprints:6.3_jack_new_ref" (at 43.18 147.32 0)
       (effects (font (size 1.27 1.27)) hide)
     )
@@
       (effects (font (size 1.27 1.27)) hide)
     )
-    (property "LCSC Part" "C309275" (at 43.18 147.32 0)
-      (effects (font (size 1.27 1.27)) hide)
-    )
+    (property "LCSC Part" "C309277" (at 43.18 147.32 0)
+      (effects (font (size 1.27 1.27)) hide)
+    )
