File: stm_audio_board_V3/Power.kicad_sch (KiCad schematic)
At the start: 125 parts, among them J5 Barrel_Jack_MountingPin, U1 IS42S16100H-7TL, U2 OP275, U20 AP1117-33, U3 7909, U4 OP275, U5 AP1117-33, U6 7809, U9 AP1117-33

Commit message: added silkscreen captions, capacitor between gnd and earth
Parts:
- removed J5: Barrel_Jack_MountingPin, Connector_BarrelJack:BarrelJack_GCT_DCJ200-10-A_Horizontal, symbol Connector:Barrel_Jack_MountingPin
- added C30: 1nF, Capacitor_THT:C_Disc_D7.5mm_W5.0mm_P7.50mm, symbol Device:C_Small
- added J3: Barrel_Jack_Switch, Connector_BarrelJack:BarrelJack_GCT_DCJ200-10-A_Horizontal, symbol Connector:Barrel_Jack_Switch
- C29, C4: footprint Capacitor_THT:CP_Radial_D6.3mm_P2.50mm -> stm_audio_board_footprints:CP_Radial_D6.3mm_P2.50mm_reference_fix
Connections:
- net Earth: now also C30.1, J3.1
- net GND: now also C30.2
- net PWR_INPUT_12V-18V: now also J3.2, J3.3
